File: board/elrs-lvs.kicad_pcb (KiCad board)
At the start: 4 copper layers, 46 x 22 mm, 85 parts, among them J1 PWM, J10 CF/Prog, J12 Balance, J13 U.FL, J2 PWM, J3 PWM, J4 PWM, J5 PWM, J6 PWM, J7 PWM, J8 PWM, J9 Little Tower, SW1 SW_SPST, SW2 SW_SPST, U1 ESP32-PICO-V3, U2 SX1281, U3 TPSM82901SISR, U4 2450FM07D0034T, Y1 52Mhz TCXO

Commit message: mess stuff up for investigating jlc pcba
Parts:
- added H1: MountingHole, elrs-lvs:MountingHole_JLC, F.Cu at (3.38, 11.0)
- added H2: MountingHole, elrs-lvs:MountingHole_JLC, B.Cu at (44.0, 2.00)
- added H3: MountingHole, elrs-lvs:MountingHole_JLC, F.Cu at (44.0, 20.0)
Routing:
- net GND: track 265.5 -> 283.5 mm
