File: board/elrs-lvs.kicad_sch (KiCad schematic)
At the start: 85 parts, among them J1 PWM, J10 CF/Prog, J12 Balance, J13 U.FL, J2 PWM, J3 PWM, J4 PWM, J5 PWM, J6 PWM, J7 PWM, J8 PWM, J9 Little Tower, SW1 SW_SPST, SW2 SW_SPST, U1 ESP32-PICO-V3, U2 SX1281, U3 TPSM82901SISR, U4 2450FM07D0034T, Y1 52Mhz TCXO

Commit message: mess stuff up for investigating jlc pcba
Parts:
- added H1, H2, H3: MountingHole, elrs-lvs:MountingHole_JLC, symbol Mechanical:MountingHole
- J1, J12, J2, J3, J4, J5, J6, J7, J8: now not fitted; now left out of the parts list
