File: board/elrs-lvs.kicad_sch (KiCad schematic)
At the start: 88 parts, among them J1 PWM, J10 CF/Prog, J12 Balance, J13 U.FL, J2 PWM, J3 PWM, J4 PWM, J5 PWM, J6 PWM, J7 PWM, J8 PWM, J9 Little Tower, SW1 SW_SPST, SW2 SW_SPST, U1 ESP32-PICO-V3, U2 SX1281, U3 TPSM82901SISR, U4 2450FM07D0034T, Y1 52Mhz TCXO

Commit message: modify design to use new regulator and switch part due to availability
Parts:
- removed C13: 470n, 10V, Capacitor_SMD:C_0402_1005Metric, symbol Device:C
- removed C6: 22u, Capacitor_SMD:C_0805_2012Metric, symbol Device:C
- removed R2: 40.2k, Resistor_SMD:R_0402_1005Metric, symbol Device:R_Small
- removed R3: 100, Resistor_SMD:R_0402_1005Metric, symbol Device:R_Small
- removed SW1: SW_SPST, elrs-lvs:SO4_SW_1563-R66-8005_MIT, symbol Switch:SW_SPST
- removed U3: TPSM82901SISR, elrs-lvs:uSIP11_SIS_TEX, symbol elrs-lvs:TPSM82901SISR
- added C13, C22, C29, C30, C31, C6: DNP, elrs-lvs:C_0805-1206, symbol Device:C_Small
- added C23, C5: 22u 25v 0603, Capacitor_SMD:C_0603_1608Metric, symbol Device:C
- added C24: 100n, Capacitor_SMD:C_0402_1005Metric, symbol Device:C
- added C25: >47u 0603, Capacitor_SMD:C_0603_1608Metric, symbol Device:C
- added C27: 10u, Capacitor_SMD:C_0402_1005Metric, symbol Device:C
- added C28: DNP, Capacitor_SMD:C_1206_3216Metric, symbol Device:C_Small
- added JP1, JP2: JP, elrs-lvs:R_0201_0603_JP, symbol Jumper:Jumper_2_Small_Bridged
- added JP3: NP, elrs-lvs:R_0201_0603_NP, symbol Jumper:Jumper_2_Small_Open
- added L2: 1-1.5uH 1A 0603, Inductor_SMD:L_0603_1608Metric, symbol Device:L
- added R49: 470k, Resistor_SMD:R_0402_1005Metric, symbol Device:R_Small
- added R5: 150k, Resistor_SMD:R_0402_1005Metric, symbol Device:R_Small
- added R6: 10k, Resistor_SMD:R_0402_1005Metric, symbol Device:R
- added U5: TPS63070RNMR, elrs-lvs:RNM0015A, symbol 2026-08-15_19-07-46:TPS63070RNMR
- C2: value 10u -> >470n; footprint Capacitor_SMD:C_0805_2012Metric -> Capacitor_SMD:C_0402_1005Metric; Digikey https://www.digikey.com/en/products/detail/murata-electroni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 -> https://www.digikey.com/en/products/detail/samsung-electro-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; LCSC C5646740 -> C318573; Manufacturer Murata -> Samsung; Part GRJ21BR61E106KE01K -> CL05A105MQ5NNNC
- SW2: footprint elrs-lvs:SO4_SW_1563-R66-8005_MIT -> elrs-lvs:SW_CK_NANOT_AS; Digikey https://www.digikey.com/en/products/detail/mitsumi-electric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 -> 108-NANOT100ASCT-ND; LCSC C4364937 -> (none); Manufacturer Mitsumi -> C&K; Part R-668048 -> NANOT 100 AS
Connections:
- net +3.3V: now also C25.1, C27.1, R49.2, U5.7 (VOUT), U5.8 (VOUT)
- net +5V: now also C13.1, C22.1, C28.1, C29.1, C30.1, C31.1, C6.1
- net GND: now also C13.2, C22.2, C23.2, C24.2, C25.2, C27.2, C28.2, C29.2, C30.2, C31.2, C5.2, C6.2, JP2.2 (B), R5.2, U5.10 (PGND), U5.15 (VSEL), U5.4 (GND), U5.6 (FB2)
- net RESET: now also JP1.1 (A)
- net V_DCC: now also C2.1
- net VIN renamed 5V_FUSED
- net 5V_FUSED: now also C23.1, C5.1, R6.1, U5.12 (VIN), U5.13 (VIN); no longer C2.1
- new net: R49.1, R5.1, U5.5 (FB)
- new net: JP3.2 (B), R6.2, U5.14 (EN)
- new net: JP2.1 (A), JP3.1 (A), U5.1 (PS_SYNC)
- new net: L2.1, U5.11 (L1)
- new net: JP1.2 (B), U5.2 (PG)
- new net: C24.1, U5.3 (VAUX)
- new net: L2.2, U5.9 (L2)
- no-connect marks 9 -> 6
Other:
- note added: "0.8v"
- note added: "1-3s 3.0-12.6v (max 2.0-16v)"
- note added: "Note: 3.3v is out of spec for led, but works. (16v from 5v input would definitely not work)"
- note added: "Optional capacitor positions for handling poor BEC and servo current spikes"
- note added: "PS Low = Forced PWM mode lower efficiency and ripple"
- note added: "TPSM82901SISR possible alt LMZ21701 expensive but small TPSM336{20,10,06) slightly larger but more available, TPSM33620S3QRDNRQ1 TPS63070 buck/boost highly available but large"
- note added: "V2: invert serial connector pinout (to match radiomaster), remove test points, re-layout for single sided and larger (cheaper) clearances (v2 never built due to part availability) V2.1: change to buck-bootst regulator (more available), remove EN button to save space"
- note removed: "1-3s 3.3-12.6v (max 3.0-17v)"
- note removed: "Discharge off 2.5Mhz (ds 7-1) FB as VSET Auto PFM"
- note removed: "Note: 3.3v is out of spec for led, but works. (17v would definitely not work)"
- note removed: "Note: chosen to have zero drop (100% duty cycle) operation to allow operation below 3.3v input"
- note removed: "V2: invert serial connector pinout (to match radiomaster), remove test points, re-layout for single sided and larger (cheaper) clearances"
- note removed: "VSET Open 3.3v (ds 7-3)"
- moved on the sheet: D1, D2, D3, F1, R14

Commit message: minor board cleanup
Parts:
- U5: Manufacturer (none) -> Texas Instruments; Part (none) -> TPS63070RNMR
Changed lines of the file:
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@@
+			)
+		)
+		(property "Manufacturer" "Texas Instruments"
+			(at 85.09 39.37 0)
+			(hide yes)
+			(show_name no)
+			(do_not_autoplace no)
+			(effects
+				(font
+					(size 1.27 1.27)
+				)
+			)
+		)
+		(property "Part" "TPS63070RNMR"
+			(at 85.09 39.37 0)
+			(hide yes)
+			(show_name no)
+			(do_not_autoplace no)
+			(effects
+				(font
+					(size 1.27 1.27)
+				)
 			)
 		)
@@
 		)
 		(property "Value" "GND"
-			(at 74.168 45.72 90)
-			(show_name no)
-			(do_not_autoplace no)
+			(at 76.454 44.45 90)
+			(show_name no)
+			(do_not_autoplace no)

Commit message: pick initial parts, prior to review
Parts:
- C13, C22, C28, C29, C30, C31, C6: value DNP -> >16v; Digikey (none) -> 587-3246-1-ND; Manufacturer (none) -> Taiyo Yuden; Part (none) -> TMK316BBJ226ML-T; now not fitted
- C23, C5: Alt part number (none) -> 0603YD226MAT2A; Digikey (none) -> 478-KGM15CR51E226MTCT-ND; Manufacturer (none) -> KYOCERA AVX; Part (none) -> KGM15CR51E226MT
- C25: Digikey (none) -> 4587-C0603B476M007TCT-ND; Manufacturer (none) -> Holy Stone Enterprise Co., Ltd.; Part (none) -> C0603B476M007T
- D1: value 17v -> 16v
- J13: Digikey (none) -> 26-U.FL-R-SMT-1(80)CT-ND
- JP1, JP2, JP3: Digikey (none) -> CR0201-J/-000GLFCT-ND; Manufacturer (none) -> Bourns; Part (none) -> CR0201-J/-000GLF; now not fitted
- L2: Digikey (none) -> 535-AOTA-B160808S1R0MTCT-ND; Manufacturer (none) -> Abracon LLC; Part (none) -> AOTA-B160808S1R0MT
- R5: Digikey (none) -> 13-RT0402FRE07150KLCT-ND; Manufacturer (none) -> Yageo; Part (none) -> RT0402FRE07150KL
- U5: Digikey (none) -> 296-44874-1-ND
Other:
- note added: "3.3v 0.5A"

Commit message: more parts picking
Parts:
- C1, C2: Digikey https://www.digikey.com/en/products/detail/samsung-electro-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 -> 1276-1235-1-ND
- C10, C11, C12, C14, C15, C16, C17, C18, C19, C20, C21, C24, C3: Alt part number (none) -> CL05A104KA5NNNC; Digikey https://www.digikey.com/en/products/detail/samsung-electro-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 -> 1292-1629-1-ND; Manufacturer Samsung -> Walsin Technology Corporation; Part CL05A104KA5NNNC -> 0402B104K100CT
- C23, C5: Alt part number 0603YD226MAT2A -> 0603YD226MAT2A CL10A106MA8NRNC; LCSC (none) -> C96446
- C25: Alt part number (none) -> GRM188R60J476ME15D; LCSC (none) -> C140782
- C27, C4: Digikey https://www.digikey.com/en/products/detail/samsung-electro-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 -> 490-GRM155R60J106ME05DCT-ND; Manufacturer Samsung -> Murata Electronics; Part CL05A106MQ5NUNC -> GRM155R60J106ME05D
- C7, C8: Digikey https://www.digikey.com/en/products/detail/samsung-electro-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 -> 1276-1028-1-ND
- C9: Digikey https://www.digikey.com/en/products/detail/kyocera-avx/KGM0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 -> 478-KGM05AR71H102KNCT-ND
- F1: LCSC C634245 -> C720078
- L2: Alt part number (none) -> LSCNB1608HKT1R0MD; LCSC (none) -> C6585190
- R5: LCSC (none) -> C25755
- U4: Alt part number 2450FM07A0029T -> 2450FM07D0034T 2450FM07A0029T 2450FM07D0034001T; LCSC C2651081 -> C6054595; Mouser 609-2450FM07D0034T -> 609-2450FM07D0034001 609-2450FM07D0034T; Part 2450FM07D0034T -> 2450FM07D0034001T
- U5: LCSC (none) -> C109322
Other:
- note added: "https://jlcpcb.com/parts"

Commit message: change 17v zener to 12v - next option down from same mfr
Parts:
- C13, C22, C28, C29, C30, C31, C6, JP1, JP2, JP3: now left out of the parts list
- D1: value 16v -> 13v; Digikey https://www.digikey.com/en/products/detail/toshiba-semicond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 -> 264-CUHZ12VH3FCT-ND; LCSC C7236804 -> C5609188; Part CUHZ16V,H3F -> CUHZ12V,H3F
- H1, H2, H3: now not fitted
- SW2: now not fitted; now left out of the parts list
Changed lines of the file:
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@@
 		(on_board yes)
 		(in_pos_files yes)
-		(dnp no)
+		(dnp yes)
 		(fields_autoplaced yes)
 		(property "Reference" "H2"
@@
 		(body_style 1)
 		(exclude_from_sim no)
-		(in_bom yes)
+		(in_bom no)
 		(on_board yes)
 		(in_pos_files yes)
@@
 		(body_style 1)
 		(exclude_from_sim no)
-		(in_bom yes)
+		(in_bom no)
 		(on_board yes)
 		(in_pos_files yes)
@@
 		(body_style 1)
 		(exclude_from_sim no)
-		(in_bom yes)
+		(in_bom no)
 		(on_board yes)
 		(in_pos_files yes)
@@
 		(body_style 1)
 		(exclude_from_sim no)
-		(in_bom yes)
+		(in_bom no)
 		(on_board yes)
 		(in_pos_files yes)
@@
 		(on_board yes)
 		(in_pos_files yes)
-		(dnp no)
+		(dnp yes)
 		(fields_autoplaced yes)
 		(property "Reference" "H1"
@@
 		(body_style 1)
 		(exclude_from_sim no)
-		(in_bom yes)
+		(in_bom no)
 		(on_board yes)
 		(in_pos_files yes)
@@
 		(on_board yes)
 		(in_pos_files yes)
-		(dnp no)
+		(dnp yes)
 		(fields_autoplaced yes)
 		(property "Reference" "H3"
@@
 		(body_style 1)
 		(exclude_from_sim no)
-		(in_bom yes)
+		(in_bom no)
 		(on_board yes)
 		(in_pos_files yes)
@@
 		(body_style 1)
 		(exclude_from_sim no)
-		(in_bom yes)
+		(in_bom no)
 		(on_board yes)
 		(in_pos_files yes)
@@
 		(body_style 1)
 		(exclude_from_sim no)
-		(in_bom yes)
+		(in_bom no)
 		(on_board yes)
 		(in_pos_files yes)
@@
 			)
 		)
-		(property "Value" "16v"
+		(property "Value" "13v"
 			(at 21.59 34.2899 90)
 			(show_name no)
@@
 			)
 		)
-		(property "Digikey" "https://www.digikey.com/en/products/detail/toshiba-semiconductor-and-storage/CUHZ16V-H3F/15857862"
+		(property "Digikey" "264-CUHZ12VH3FCT-ND"
 			(at 19.05 33.02 0)
 			(hide yes)
@@
 			)
 		)
-		(property "Part" "CUHZ16V,H3F"
+		(property "Part" "CUHZ12V,H3F"
 			(at 19.05 33.02 0)
 			(hide yes)
@@
 			)
 		)
-		(property "LCSC" "C7236804"
+		(property "LCSC" "C5609188"
 			(at 19.05 33.02 90)
 			(hide yes)
@@
 		(body_style 1)
 		(exclude_from_sim no)
-		(in_bom yes)
+		(in_bom no)
 		(on_board yes)
 		(in_pos_files yes)
-		(dnp no)
+		(dnp yes)
 		(fields_autoplaced yes)
 		(property "Reference" "SW2"
@@
 		(body_style 1)
 		(exclude_from_sim no)
-		(in_bom yes)
+		(in_bom no)
 		(on_board yes)
 		(in_pos_files yes)
@@
 		(body_style 1)
 		(exclude_from_sim no)
-		(in_bom yes)
+		(in_bom no)
 		(on_board yes)
 		(in_pos_files yes)
